File: 5pin_version.kicad_sch (KiCad schematic)
At the start: 4 parts

Commit message: completed re-routing
Changed lines of the file:
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@@
 			)
 		)
-		(pin "COL4" input
+		(pin "COL4" output
 			(at 184.15 87.63 180)
 			(effects
@@
 			)
 		)
-		(pin "COL1" input
+		(pin "COL1" output
 			(at 184.15 80.01 180)
 			(effects
@@
 			)
 		)
-		(pin "ROW1" output
+		(pin "ROW1" input
 			(at 184.15 69.85 180)
 			(effects
@@
 			)
 		)
-		(pin "ROW0" output
+		(pin "ROW0" input
 			(at 184.15 67.31 180)
 			(effects
@@
 			)
 		)
-		(pin "ROW2" output
+		(pin "ROW2" input
 			(at 184.15 72.39 180)
 			(effects
@@
 			)
 		)
-		(pin "COL0" input
+		(pin "COL0" output
 			(at 184.15 77.47 180)
 			(effects
@@
 			)
 		)
-		(pin "COL2" input
+		(pin "COL2" output
 			(at 184.15 82.55 180)
 			(effects
@@
 			)
 		)
-		(pin "COL3" input
+		(pin "COL3" output
 			(at 184.15 85.09 180)
 			(effects
@@
 			)
 		)
-		(pin "COL9" input
+		(pin "COL9" output
 			(at 184.15 100.33 180)
 			(effects
@@
 			)
 		)
-		(pin "COL5" input
+		(pin "COL5" output
 			(at 184.15 90.17 180)
 			(effects
@@
 			)
 		)
-		(pin "COL6" input
+		(pin "COL6" output
 			(at 184.15 92.71 180)
 			(effects
@@
 			)
 		)
-		(pin "COL7" input
+		(pin "COL7" output
 			(at 184.15 95.25 180)
 			(effects
@@
 			)
 		)
-		(pin "COL8" input
+		(pin "COL8" output
 			(at 184.15 97.79 180)
 			(effects
@@
 			)
 		)
-		(pin "ROW2" input
+		(pin "ROW2" output
 			(at 142.24 72.39 0)
 			(effects
@@
 			)
 		)
-		(pin "COL2" output
+		(pin "COL2" input
 			(at 142.24 82.55 0)
 			(effects
@@
 			)
 		)
-		(pin "COL0" output
+		(pin "COL0" input
 			(at 142.24 77.47 0)
 			(effects
@@
 			)
 		)
-		(pin "COL1" output
+		(pin "COL1" input
 			(at 142.24 80.01 0)
 			(effects
@@
 			)
 		)
-		(pin "COL3" output
+		(pin "COL3" input
 			(at 142.24 85.09 0)
 			(effects
@@
 			)
 		)
-		(pin "COL4" output
+		(pin "COL4" input
 			(at 142.24 87.63 0)
 			(effects
@@
 			)
 		)
-		(pin "ROW0" input
+		(pin "ROW0" output
 			(at 142.24 67.31 0)
 			(effects
@@
 			)
 		)
-		(pin "ROW1" input
+		(pin "ROW1" output
 			(at 142.24 69.85 0)
 			(effects
@@
 			)
 		)
-		(pin "COL6" output
+		(pin "COL6" input
 			(at 142.24 92.71 0)
 			(effects
@@
 			)
 		)
-		(pin "COL7" output
+		(pin "COL7" input
 			(at 142.24 95.25 0)
 			(effects
@@
 			)
 		)
-		(pin "COL5" output
+		(pin "COL5" input
 			(at 142.24 90.17 0)
 			(effects
@@
 			)
 		)
-		(pin "COL9" output
+		(pin "COL9" input
 			(at 142.24 100.33 0)
 			(effects
@@
 			)
 		)
-		(pin "COL8" output
+		(pin "COL8" input
 			(at 142.24 97.79 0)
 			(effects
