File: matrix.kicad_sch (KiCad schematic)
At the start: 60 parts, among them SW1 SW_Push, SW10 SW_Push, SW11 SW_Push, SW12 SW_Push, SW13 SW_Push, SW14 SW_Push, SW15 SW_Push, SW16 SW_Push, SW17 SW_Push, SW18 SW_Push, SW19 SW_Push, SW2 SW_Push, SW20 SW_Push, SW21 SW_Push, SW22 SW_Push, SW23 SW_Push, SW24 SW_Push, SW25 SW_Push, SW26 SW_Push, SW27 SW_Push, SW28 SW_Push, SW29 SW_Push, SW3 SW_Push, SW30 SW_Push, SW4 SW_Push, SW5 SW_Push, SW6 SW_Push, SW7 SW_Push, SW8 SW_Push, SW9 SW_Push

Commit message: completed re-routing
Connections:
- net ROW0: now also D1.2 (A), D10.2 (A), D2.2 (A), D3.2 (A), D4.2 (A), D5.2 (A), D6.2 (A), D7.2 (A), D8.2 (A), D9.2 (A); no longer D1.1 (K), D10.1 (K), D2.1 (K), D3.1 (K), D4.1 (K), D5.1 (K), D6.1 (K), D7.1 (K), D8.1 (K), D9.1 (K)
- net ROW1: now also D11.2 (A), D12.2 (A), D13.2 (A), D14.2 (A), D15.2 (A), D16.2 (A), D17.2 (A), D18.2 (A), D19.2 (A), D20.2 (A); no longer D11.1 (K), D12.1 (K), D13.1 (K), D14.1 (K), D15.1 (K), D16.1 (K), D17.1 (K), D18.1 (K), D19.1 (K), D20.1 (K)
- net ROW2: now also D21.2 (A), D22.2 (A), D23.2 (A), D24.2 (A), D25.2 (A), D26.2 (A), D27.2 (A), D28.2 (A), D29.2 (A), D30.2 (A); no longer D21.1 (K), D22.1 (K), D23.1 (K), D24.1 (K), D25.1 (K), D26.1 (K), D27.1 (K), D28.1 (K), D29.1 (K), D30.1 (K)
- net at SW16.1: now also D16.1 (K); no longer D16.2 (A)
- net at SW24.1: now also D24.1 (K); no longer D24.2 (A)
- net at SW23.1: now also D23.1 (K); no longer D23.2 (A)
- net at SW4.1: now also D4.1 (K); no longer D4.2 (A)
- net at SW11.1: now also D11.1 (K); no longer D11.2 (A)
- net at SW20.1: now also D20.1 (K); no longer D20.2 (A)
- net at SW18.1: now also D18.1 (K); no longer D18.2 (A)
- net at SW13.1: now also D13.1 (K); no longer D13.2 (A)
- net at SW30.1: now also D30.1 (K); no longer D30.2 (A)
- net at SW28.1: now also D28.1 (K); no longer D28.2 (A)
- net at SW26.1: now also D26.1 (K); no longer D26.2 (A)
- net at SW6.1: now also D6.1 (K); no longer D6.2 (A)
- net at SW9.1: now also D9.1 (K); no longer D9.2 (A)
- net at SW17.1: now also D17.1 (K); no longer D17.2 (A)
- net at SW25.1: now also D25.1 (K); no longer D25.2 (A)
- net at SW22.1: now also D22.1 (K); no longer D22.2 (A)
- net at SW29.1: now also D29.1 (K); no longer D29.2 (A)
- net at SW27.1: now also D27.1 (K); no longer D27.2 (A)
- net at SW8.1: now also D8.1 (K); no longer D8.2 (A)
- net at SW19.1: now also D19.1 (K); no longer D19.2 (A)
- net at SW5.1: now also D5.1 (K); no longer D5.2 (A)
- net at SW2.1: now also D2.1 (K); no longer D2.2 (A)
- net at SW14.1: now also D14.1 (K); no longer D14.2 (A)
- net at SW10.1: now also D10.1 (K); no longer D10.2 (A)
- net at SW15.1: now also D15.1 (K); no longer D15.2 (A)
- net at SW1.1: now also D1.1 (K); no longer D1.2 (A)
- net at SW12.1: now also D12.1 (K); no longer D12.2 (A)
- net at SW21.1: now also D21.1 (K); no longer D21.2 (A)
- net at SW3.1: now also D3.1 (K); no longer D3.2 (A)
- net at SW7.1: now also D7.1 (K); no longer D7.2 (A)
