File: mcu.kicad_sch (KiCad schematic)
At the start: 10 parts, among them J3 Conn_01x04_Pin, U2 STM32L053C8T6

Commit message: rewired most lines, changed sizes to make easier to solder
Parts:
- C12, C3, C4, C6, C7, C8, C9: footprint Capacitor_SMD:C_0402_1005Metric -> Capacitor_SMD:C_0603_1608Metric
Changed lines of the file:
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@@
 			)
 		)
-		(property "Footprint" "Capacitor_SMD:C_0402_1005Metric"
+		(property "Footprint" "Capacitor_SMD:C_0603_1608Metric"
 			(at 116.5352 66.04 0)
 			(effects
@@
 			)
 		)
-		(property "Footprint" "Capacitor_SMD:C_0402_1005Metric"
+		(property "Footprint" "Capacitor_SMD:C_0603_1608Metric"
 			(at 176.2252 66.04 0)
 			(effects
@@
 			)
 		)
-		(property "Footprint" "Capacitor_SMD:C_0402_1005Metric"
+		(property "Footprint" "Capacitor_SMD:C_0603_1608Metric"
 			(at 176.2252 44.45 0)
 			(effects
@@
 			)
 		)
-		(property "Footprint" "Capacitor_SMD:C_0402_1005Metric"
+		(property "Footprint" "Capacitor_SMD:C_0603_1608Metric"
 			(at 92.4052 83.82 0)
 			(effects
@@
 			)
 		)
-		(property "Footprint" "Capacitor_SMD:C_0402_1005Metric"
+		(property "Footprint" "Capacitor_SMD:C_0603_1608Metric"
 			(at 127.9652 66.04 0)
 			(effects
@@
 			)
 		)
-		(property "Footprint" "Capacitor_SMD:C_0402_1005Metric"
+		(property "Footprint" "Capacitor_SMD:C_0603_1608Metric"
 			(at 186.3852 44.45 0)
 			(effects
@@
 			)
 		)
-		(property "Footprint" "Capacitor_SMD:C_0402_1005Metric"
+		(property "Footprint" "Capacitor_SMD:C_0603_1608Metric"
 			(at 186.3852 66.04 0)
 			(effects

Commit message: completed re-routing
Connections:
- net COL0: now also U2.39 (PB3); no longer U2.2 (PC13)
- net COL1: now also U2.40 (PB4); no longer U2.42 (PB6)
- net COL3: now also U2.42 (PB6); no longer U2.4 (PC15)
- net COL4: now also U2.43 (PB7); no longer U2.3 (PC14)
- net COL5: now also U2.13 (PA3); no longer U2.26 (PB13)
- net COL6: now also U2.17 (PA7); no longer U2.25 (PB12)
- net COL7: now also U2.16 (PA6); no longer U2.27 (PB14)
- net COL8: now also U2.15 (PA5); no longer U2.28 (PB15)
- net COL9: now also U2.14 (PA4); no longer U2.29 (PA8)
- net ROW0: now also U2.3 (PC14); no longer U2.16 (PA6)
- net ROW1: now also U2.2 (PC13); no longer U2.17 (PA7)
